File: mulletpad-pcb.kicad_pcb (KiCad board)
At the start: 2 copper layers, 73.4 x 98.1 mm, 56 parts, among them SW0 KEYSW, SW1 KEYSW, SW10 KEYSW, SW11 KEYSW, SW12 KEYSW, SW13 KEYSW, SW14 KEYSW, SW15 KEYSW, SW16 KEYSW, SW2 KEYSW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

Commit message: clean up gnd fills
Routing:
- net GND: track 179.4 -> 180.8 mm
Changed lines of the file:
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@@
     (thickness 1.6)
     (drawings 540)
-    (tracks 596)
+    (tracks 594)
     (zones 0)
     (modules 56)
@@
   (segment (start 164.250597 63.201572) (end 164.054601 63.397568) (width 0.25) (layer B.Cu) (net 2))
   (via (at 164.054601 63.397568) (size 0.8) (drill 0.4) (layers F.Cu B.Cu) (net 2))
-  (segment (start 178.726156 58.674559) (end 177.333969 58.674559) (width 0.25) (layer B.Cu) (net 2))
-  (segment (start 176.691438 60.901992) (end 176.314435 61.278995) (width 0.25) (layer B.Cu) (net 2))
-  (segment (start 177.333969 58.674559) (end 177.163875 58.844653) (width 0.25) (layer B.Cu) (net 2))
-  (segment (start 177.163875 58.844653) (end 177.163875 59.579555) (width 0.25) (layer B.Cu) (net 2))
-  (segment (start 177.163875 59.579555) (end 176.691438 60.051992) (width 0.25) (layer B.Cu) (net 2))
-  (segment (start 176.691438 60.051992) (end 176.691438 60.901992) (width 0.25) (layer B.Cu) (net 2))
   (segment (start 177.858783 55.472496) (end 178.213735 55.117544) (width 0.25) (layer B.Cu) (net 2))
   (segment (start 175.954183 55.472496) (end 177.858783 55.472496) (width 0.25) (layer B.Cu) (net 2))
-  (segment (start 178.213735 55.117544) (end 178.788735 55.117544) (width 0.25) (layer B.Cu) (net 2))
   (segment (start 179.526166 65.09132) (end 179.526166 59.474569) (width 0.25) (layer B.Cu) (net 2))
   (segment (start 177.268861 72.86039) (end 177.843861 72.86039) (width 0.25) (layer B.Cu) (net 2))
@@
   (segment (start 174.736582 72.16526) (end 175.431712 72.86039) (width 0.25) (layer B.Cu) (net 2))
   (segment (start 179.013745 58.936918) (end 179.00113 58.949533) (width 0.25) (layer B.Cu) (net 2))
-  (segment (start 179.013745 55.342554) (end 179.013745 58.936918) (width 0.25) (layer B.Cu) (net 2))
-  (segment (start 178.998813 55.327622) (end 179.013745 55.342554) (width 0.25) (layer B.Cu) (net 2))
-  (segment (start 178.788735 55.117544) (end 178.998813 55.327622) (width 0.25) (layer B.Cu) (net 2))
   (segment (start 179.526166 59.474569) (end 179.00113 58.949533) (width 0.25) (layer B.Cu) (net 2))
-  (segment (start 179.00113 58.949533) (end 178.726156 58.674559) (width 0.25) (layer B.Cu) (net 2))
   (segment (start 168.449573 67.979005) (end 167.820121 68.608457) (width 0.25) (layer B.Cu) (net 2))
   (segment (start 170.687447 67.979005) (end 168.449573 67.979005) (width 0.25) (layer B.Cu) (net 2))
   (segment (start 170.964435 67.128995) (end 170.964435 67.702017) (width 0.25) (layer B.Cu) (net 2))
   (segment (start 170.964435 67.702017) (end 170.687447 67.979005) (width 0.25) (layer B.Cu) (net 2))
+  (segment (start 178.726156 58.674559) (end 179.00113 58.949533) (width 0.25) (layer B.Cu) (net 2))
+  (segment (start 176.813523 58.674559) (end 178.726156 58.674559) (width 0.25) (layer B.Cu) (net 2))
+  (segment (start 176.314435 59.173647) (end 176.813523 58.674559) (width 0.25) (layer B.Cu) (net 2))
+  (segment (start 176.314435 61.278995) (end 176.314435 59.173647) (width 0.25) (layer B.Cu) (net 2))
+  (segment (start 179.526166 58.899569) (end 179.529479 58.896256) (width 0.25) (layer B.Cu) (net 2))
+  (segment (start 179.526166 59.474569) (end 179.526166 58.899569) (width 0.25) (layer B.Cu) (net 2))
+  (segment (start 179.529479 58.896256) (end 179.529479 55.328675) (width 0.25) (layer B.Cu) (net 2))
+  (segment (start 179.318348 55.117544) (end 178.213735 55.117544) (width 0.25) (layer B.Cu) (net 2))
+  (segment (start 179.529479 55.328675) (end 179.318348 55.117544) (width 0.25) (layer B.Cu) (net 2))
   (segment (start 173.419181 55.472496) (end 172.464435 56.427242) (width 0.25) (layer B.Cu) (net 3))
   (segment (start 173.754183 55.472496) (end 173.419181 55.472496) (width 0.25) (layer B.Cu) (net 3))
@@
     (polygon
       (pts
-        (xy 180.470934 58.949639) (xy 178.528693 58.975886) (xy 177.531326 58.897146) (xy 177.478833 59.422076) (xy 177.301669 61.101852)
-        (xy 173.909309 61.101852) (xy 170.808627 58.162244) (xy 169.867348 58.162244) (xy 169.867348 53.490367) (xy 180.365948 53.490367)
+        (xy 180.404379 58.198347) (xy 177.202316 61.100373) (xy 172.932733 61.120513) (xy 172.932733 58.163351) (xy 170.808627 58.162244)
+        (xy 168.138281 58.145853) (xy 168.120783 56.693519) (xy 167.175891 55.818619) (xy 164.988641 55.818619) (xy 164.953645 44.514911)
+        (xy 180.526865 44.567405)
       )
     )
