File: mulletpad-pcb.kicad_pcb (KiCad board)
At the start: 2 copper layers, 73.4 x 98.1 mm, 56 parts, among them SW0 KEYSW, SW1 KEYSW, SW10 KEYSW, SW11 KEYSW, SW12 KEYSW, SW13 KEYSW, SW14 KEYSW, SW15 KEYSW, SW16 KEYSW, SW2 KEYSW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

Commit message: Update mulletpad-pcb.kicad_pcb
Parts:
- moved C8 0.32 mm to (167.9, 68.1)
- moved D13 0.25 mm to (150.2, 114.1)
- moved D9 0.25 mm to (131.1, 114.1)
- moved D11 0.21 mm to (145.4, 70.6)
- moved D7 0.16 mm to (142.4, 70.6)
- moved D5 0.13 mm to (121.5, 133.1)
- moved D12 0.13 mm to (150.2, 95.9)
- moved D8 0.13 mm to (131.4, 95.9)
- turned C6 to 180 degrees
Routing:
- net GND: track 180.8 -> 87.3 mm, vias 4 -> 10
- net row4: track 223.0 -> 253.3 mm, vias 0 -> 2
- net col3: track 85.0 -> 106.4 mm
- net Net-(D2-Pad2): track 23.8 -> 12.3 mm, vias 2 -> 0
- net row2: track 169.5 -> 160.2 mm, vias 2 -> 0
- net row3: track 165.0 -> 156.3 mm
- net row1: track 86.6 -> 80.6 mm
- net col2: track 120.4 -> 115.7 mm
- net +5V: track 99.9 -> 102.3 mm, vias 4 -> 6
- net row0: track 160.2 -> 161.5 mm
- net D+: track 12.2 -> 11.4 mm
- net Net-(D16-Pad2): track 9.49 -> 8.73 mm
- net col1: track 113.1 -> 112.4 mm
- net Net-(R3-Pad1): track 65.4 -> 64.9 mm
- added copper zone on F.Cu, net GND
